File: Mods/anchit92/PCB_version/PCB_files/seeed_studio_GNSS/seeed_studio_GNSS.kicad_pcb (KiCad board)
At the start: 2 copper layers, 47.5 x 21 mm, 11 parts, among them Q1 AO3401A, U1 SAM-M10Q-00B, U2 XIAO-nRF52840-SMD

Commit message: Updated PCB based on experience
Parts:
- removed R6: 0, Resistor_SMD:R_0402_1005Metric
- added JP1: SolderJumper_2_Bridged, Jumper:SolderJumper-2_P1.3mm_Bridged_Pad1.0x1.5mm, B.Cu at (182.2, 101.0)
Routing:
- net +3.3V: track 55.6 -> 54.7 mm
- net Net-(JP1-A): track 3.23 -> 3.84 mm
Other:
- board text added: "v1.1"
Changed lines of the file:
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@@
 	(net 29 "Net-(Q1-D)")
 	(net 30 "Net-(Q1-G)")
-	(net 31 "Net-(U1-V_BCKP)")
+	(net 31 "Net-(JP1-A)")
 	(footprint "Resistor_SMD:R_0603_1608Metric"
 		(layer "F.Cu")
@@
 		(at 179.1354 101 180)
 		(property "Reference" "U1"
-			(at -0.3646 0.75 0)
+			(at 1.3854 0.75 0)
 			(layer "F.SilkS")
 			(effects
@@
 			(size 3.8 1.5)
 			(layers "F.Cu")
-			(net 31 "Net-(U1-V_BCKP)")
+			(net 31 "Net-(JP1-A)")
 			(pinfunction "V_BCKP")
 			(pintype "power_in")
@@
 		(embedded_fonts no)
 	)
-	(footprint "Resistor_SMD:R_0402_1005Metric"
+	(footprint "Jumper:SolderJumper-2_P1.3mm_Bridged_Pad1.0x1.5mm"
 		(layer "B.Cu")
-		(at 183 101 180)
-		(descr "Resistor SMD 0402 (1005 Metric), square (rectangular) end terminal, IPC-7351 nominal, (Body size source: IPC-SM-782 page 72, https://www.pcb-3d.com/wordpress/wp-content/uploads/ipc-sm-782a_amendment_1_and_2.pdf), generated with kicad-footprint-generator")
-		(tags "resistor")
-		(property "Reference" "R6"
-			(at 0 1.17 0)
+		(at 182.25 101 180)
+		(descr "SMD Solder Jumper, 1x1.5mm Pads, 0.3mm gap, bridged with 1 copper strip")
+		(tags "net tie solder jumper bridged")
+		(property "Reference" "JP1"
+			(at 0 1.8 0)
 			(layer "B.SilkS")
 			(hide yes)
@@
 			)
 		)
-		(property "Value" "0"
-			(at 0 -1.17 0)
+		(property "Value" "SolderJumper_2_Bridged"
+			(at 0 -1.9 0)
 			(layer "B.Fab")
 			(effects
@@
 		(property "Datasheet" "~"
 			(at 0 0 0)
+			(unlocked yes)
 			(layer "B.Fab")
 			(hide yes)
@@
 			)
 		)
-		(property "Description" "Resistor"
+		(property "Description" "Solder Jumper, 2-pole, closed/bridged"
 			(at 0 0 0)
+			(unlocked yes)
 			(layer "B.Fab")
 			(hide yes)
@@
 			)
 		)
-		(property ki_fp_filters "R_*")
+		(property ki_fp_filters "SolderJumper*Bridged*")
 		(sheetname "/")
 		(sheetfile "seeed_studio_GNSS.kicad_sch")
-		(attr smd exclude_from_bom dnp)
-		(fp_line
-			(start -0.153641 0.38)
-			(end 0.153641 0.38)
+		(zone_connect 1)
+		(attr exclude_from_pos_files exclude_from_bom allow_soldermask_bridges)
+		(net_tie_pad_groups "1, 2")
+		(fp_poly
+			(pts
+				(xy -0.25 0.3) (xy 0.25 0.3) (xy 0.25 -0.3) (xy -0.25 -0.3)
+			)
 			(stroke
-				(width 0.12)
+				(width 0)
 				(type solid)
 			)
-			(layer "B.SilkS")
+			(fill yes)
+			(layer "B.Cu")
+		)
+		(fp_rect
+			(start -0.15 0.75)
+			(end 0.15 -0.75)
+			(stroke
+				(width 0)
+				(type default)
+			)
+			(fill yes)
+			(layer "B.Mask")
 		)
 		(fp_line
-			(start -0.153641 -0.38)
-			(end 0.153641 -0.38)
+			(start 1.4 1)
+			(end 1.4 -1)
 			(stroke
 				(width 0.12)
@@
 		)
 		(fp_line
-			(start 0.93 0.47)
-			(end 0.93 -0.47)
+			(start 1.4 -1)
+			(end -1.4 -1)
 			(stroke
-				(width 0.05)
+				(width 0.12)
 				(type solid)
 			)
-			(layer "B.CrtYd")
+			(layer "B.SilkS")
 		)
 		(fp_line
-			(start 0.93 -0.47)
-			(end -0.93 -0.47)
+			(start -1.4 1)
+			(end 1.4 1)
 			(stroke
-				(width 0.05)
+				(width 0.12)
 				(type solid)
 			)
-			(layer "B.CrtYd")
+			(layer "B.SilkS")
 		)
 		(fp_line
-			(start -0.93 0.47)
-			(end 0.93 0.47)
+			(start -1.4 -1)
+			(end -1.4 1)
 			(stroke
-				(width 0.05)
+				(width 0.12)
 				(type solid)
 			)
-			(layer "B.CrtYd")
+			(layer "B.SilkS")
 		)
 		(fp_line
-			(start -0.93 -0.47)
-			(end -0.93 0.47)
+			(start 1.65 -1.25)
+			(end 1.65 1.25)
 			(stroke
 				(width 0.05)
@@
 		)
 		(fp_line
-			(start 0.525 0.27)
-			(end 0.525 -0.27)
-			(stroke
-				(width 0.1)
-				(type solid)
-			)
-			(layer "B.Fab")
-		)
-		(fp_line
-			(start 0.525 -0.27)
-			(end -0.525 -0.27)
+			(start 1.65 -1.25)
+			(end -1.65 -1.25)
 			(stroke
-				(width 0.1)
+				(width 0.05)
 				(type solid)
 			)
-			(layer "B.Fab")
+			(layer "B.CrtYd")
 		)
 		(fp_line
-			(start -0.525 0.27)
-			(end 0.525 0.27)
+			(start -1.65 1.25)
+			(end 1.65 1.25)
 			(stroke
-				(width 0.1)
+				(width 0.05)
 				(type solid)
 			)
-			(layer "B.Fab")
+			(layer "B.CrtYd")
 		)
 		(fp_line
-			(start -0.525 -0.27)
-			(end -0.525 0.27)
+			(start -1.65 1.25)
+			(end -1.65 -1.25)
 			(stroke
-				(width 0.1)
+				(width 0.05)
 				(type solid)
 			)
-			(layer "B.Fab")
-		)
-		(fp_text user "${REFERENCE}"
-			(at 0 0 0)
-			(layer "B.Fab")
-			(effects
-				(font
-					(size 0.26 0.26)
-					(thickness 0.04)
-				)
-				(justify mirror)
-			)
+			(layer "B.CrtYd")
 		)
-		(pad "1" smd roundrect
-			(at -0.51 0 180)
-			(size 0.54 0.64)
-			(layers "B.Cu" "B.Mask" "B.Paste")
-			(roundrect_rratio 0.25)
-			(net 31 "Net-(U1-V_BCKP)")
+		(pad "1" smd rect
+			(at -0.65 0 180)
+			(size 1 1.5)
+			(layers "B.Cu" "B.Mask")
+			(net 31 "Net-(JP1-A)")
+			(pinfunction "A")
 			(pintype "passive")
 		)
-		(pad "2" smd roundrect
-			(at 0.51 0 180)
-			(size 0.54 0.64)
-			(layers "B.Cu" "B.Mask" "B.Paste")
-			(roundrect_rratio 0.25)
+		(pad "2" smd rect
+			(at 0.65 0 180)
+			(size 1 1.5)
+			(layers "B.Cu" "B.Mask")
 			(net 5 "+3.3V")
+			(pinfunction "B")
 			(pintype "passive")
 		)
 		(embedded_fonts no)
-		(model "${KICAD9_3DMODEL_DIR}/Resistor_SMD.3dshapes/R_0402_1005Metric.step"
-			(offset
-				(xyz 0 0 0)
-			)
-			(scale
-				(xyz 1 1 1)
-			)
-			(rotate
-				(xyz 0 0 0)
-			)
-		)
 	)
 	(gr_line
@@
 		)
 	)
+	(gr_text "v1.1"
+		(at 172.75 94.25 180)
+		(layer "B.SilkS")
+		(effects
+			(font
+				(size 1 1)
+				(thickness 0.1)
+			)
+			(justify left bottom mirror)
+		)
+	)
 	(gr_text "github.com/anchit92"
 		(at 170.75 91.75 180)
@@
 	)
 	(gr_text "V_BKP"
-		(at 180.75 101.5 180)
+		(at 180 102.5 180)
 		(layer "B.SilkS")
 		(effects
@@
 	)
 	(segment
-		(start 178.4121 101)
-		(end 181.5 101)
-		(width 0.2)
-		(layer "F.Cu")
-		(net 5)
-	)
-	(segment
 		(start 169.698 91.198)
 		(end 151.3046 91.198)
@@
 		(net 5)
 	)
+	(segment
+		(start 178.4121 101)
+		(end 179.75 101)
+		(width 0.2)
+		(layer "F.Cu")
+		(net 5)
+	)
 	(via
-		(at 181.5 101)
+		(at 179.75 101)
 		(size 0.6)
 		(drill 0.3)
@@
 	)
 	(segment
-		(start 181.5 101)
-		(end 182.49 101)
+		(start 179.75 101)
+		(end 181.6 101)
 		(width 0.2)
 		(layer "B.Cu")
@@
 	(segment
 		(start 184.5 101)
-		(end 183.51 101)
+		(end 182.9 101)
 		(width 0.2)
 		(layer "B.Cu")
